File: Sally-2/Sally2/Sally2.kicad_pcb (KiCad board)
At the start: 2 copper layers, 220 x 150 mm, 103 parts, among them J1 Power SW, J10 GND +5V, J11 A16, J12 Drive 1-4, J13 OPT, J14 Special_Func, J15 TX GND RX, J16 + RI -, J17 RS232, J18 IN RDY CMD OUT GND, J19 Centronics, J2 Power LED, J3 USB_B, J4 PowerUSB, J5 GND +5V, J6 Barrel_Jack, J7 GND +5V, J8 PowerBarrel, J9 - A14 +, SW1 Reset, U1 GAL16V8 - IO decoder, U10 MAX232, U11 74LS06, U12 74LS06, U13 Z84C30, U14 74LS244, U15 74LS273, U16 74LS244, U2 Z80ACPU, U3 GAL16V8 - ADR decoder, U4 27C256, U5 628128_DIP32_SSOP32, U6 GAL16V8 - glue logic, U7 74LS259, U8 74LS273, U9 WD1772_PHY, X1 16Mhz

Commit message: workover part 1
Parts:
- removed REF1, REF10, REF12, REF13, REF14, REF2, REF3, REF4, REF6, REF7, REF8, REF9, Ref11, Ref5: PinSocket_2x40_P2.54mm_Vertical, Connector_PinSocket_2.54mm:PinSocket_2x40_P2.54mm_Vertical
- removed REF15: PinSocket_2x29_P2.54mm_Vertical, Connector_PinSocket_2.54mm:PinSocket_2x29_P2.54mm_Vertical
- removed REF16: PinSocket_2x27_P2.54mm_Vertical, Connector_PinSocket_2.54mm:PinSocket_2x27_P2.54mm_Vertical
- removed REF17: PinSocket_2x25_P2.54mm_Vertical, Connector_PinSocket_2.54mm:PinSocket_2x25_P2.54mm_Vertical
- removed REF18: PinSocket_2x23_P2.54mm_Vertical, Connector_PinSocket_2.54mm:PinSocket_2x23_P2.54mm_Vertical
- removed REF19: PinSocket_2x21_P2.54mm_Vertical, Connector_PinSocket_2.54mm:PinSocket_2x21_P2.54mm_Vertical
- removed REF20, REF21: PinSocket_2x14_P2.54mm_Vertical, Connector_PinSocket_2.54mm:PinSocket_2x14_P2.54mm_Vertical
- removed REF22: PinSocket_1x14_P2.54mm_Vertical, Connector_PinSocket_2.54mm:PinSocket_1x14_P2.54mm_Vertical
- removed REF23, REF24: PinSocket_2x34_P2.54mm_Vertical, Connector_PinSocket_2.54mm:PinSocket_2x34_P2.54mm_Vertical
- removed REF25, REF26: PinSocket_1x34_P2.54mm_Vertical, Connector_PinSocket_2.54mm:PinSocket_1x34_P2.54mm_Vertical
- removed SIO1: SIO 1, TF_Atari:SIO
- removed SIO2: SIO 2, TF_Atari:SIO
- added J20: Conn_01x13, Sally2:SIO_JACK, F.Cu at (154.2, 9.50)
- J16: value + RI - -> - RI +
- J4: value PowerUSB -> PowerIn
- J8: value PowerBarrel -> Conn_01x13; footprint Connector_PinHeader_2.54mm:PinHeader_1x02_P2.54mm_Vertical -> Sally2:SIO_JACK
- J9: value - A14 + -> + A14 -
- moved J8 169.7 mm to (203.5, 9.50), turned to 180 degrees
- moved X1 96.8 mm to (102.8, 101.0)
- moved C3 36.4 mm to (184.5, 82.0)
- moved U9 34.2 mm to (145.3, 93.0)
- moved U3 6.72 mm to (75.1, 101.1)
- moved U6 5.37 mm to (145.2, 47.6)
- moved U16 4.64 mm to (113.8, 47.5)
- moved U14 4.33 mm to (113.8, 66.0)
- moved U1 0.72 mm to (47.1, 101.3)
Connections:
- J6 pad 1: Net-(J8-Pin_2) -> Net-(J1-Pin_2)
- J6 pad 2: Net-(J8-Pin_1) -> GND
- J8 pad 1: Net-(J8-Pin_1) -> /SIO1
- J8 pad 2: Net-(J8-Pin_2) -> /SIO2
- U1 pad 8: unconnected-(U1-I8-Pad8) -> M1\
- U12 pad 3: unconnected-(U12-Pad3) -> Net-(U9-STEP)
- U13 pad 1: /IO/D4 -> D4
- U13 pad 15: M1\ -> CLK4
- U13 pad 18: /IO/A0 -> A0
- U13 pad 19: /IO/A1 -> A1
- U13 pad 2: /IO/D5 -> D5
- U13 pad 25: /IO/D0 -> D0
- U13 pad 26: /IO/D1 -> D1
- U13 pad 27: /IO/D2 -> D2
- U13 pad 28: /IO/D3 -> D3
- U13 pad 3: /IO/D6 -> D6
- U13 pad 4: /IO/D7 -> D7
- U14 pad 12: /IO/D1 -> D1
- U14 pad 14: /IO/D2 -> D2
- U14 pad 16: /IO/D3 -> D3
- U14 pad 18: /IO/D7 -> D7
- U15 pad 13: /IO/D4 -> D4
- U15 pad 14: /IO/D5 -> D5
- U15 pad 17: /IO/D6 -> D6
- U15 pad 18: /IO/D7 -> D7
- U15 pad 3: /IO/D0 -> D0
- U15 pad 4: /IO/D1 -> D1
- U15 pad 7: /IO/D2 -> D2
- U15 pad 8: /IO/D3 -> D3
- U16 pad 12: /IO/D3 -> D3
- U16 pad 16: /IO/D1 -> D1
- U16 pad 18: /IO/D7 -> D7
- U16 pad 3: /IO/D7 -> D7
- U16 pad 5: /IO/D6 -> D6
- U16 pad 7: /IO/D5 -> D5
- U16 pad 9: /IO/D4 -> D4
- U2 pad 10: /D6 -> D6
- U2 pad 12: /D2 -> D2
- U2 pad 13: /D7 -> D7
- U2 pad 14: /D0 -> D0
- U2 pad 15: /D1 -> D1
- U2 pad 30: /A0 -> A0
- U2 pad 31: /A1 -> A1
- U2 pad 7: /D4 -> D4
- U2 pad 8: /D3 -> D3
- U2 pad 9: /D5 -> D5
- U3 pad 11: unconnected-(U3-I10/~{OE}-Pad11) -> GND
- U3 pad 9: unconnected-(U3-I9-Pad9) -> CLK16
- U4 pad 10: /A0 -> A0
- U4 pad 11: /D0 -> D0
- U4 pad 12: /D1 -> D1
- U4 pad 13: /D2 -> D2
- U4 pad 15: /D3 -> D3
- U4 pad 16: /D4 -> D4
- U4 pad 17: /D5 -> D5
- U4 pad 18: /D6 -> D6
- U4 pad 19: /D7 -> D7
- U4 pad 9: /A1 -> A1
- U5 pad 11: /A1 -> A1
- U5 pad 12: /A0 -> A0
- U5 pad 13: /D0 -> D0
- U5 pad 14: /D1 -> D1
- U5 pad 15: /D2 -> D2
- U5 pad 17: /D3 -> D3
- U5 pad 18: /D4 -> D4
- U5 pad 19: /D5 -> D5
- U5 pad 20: /D6 -> D6
- U5 pad 21: /D7 -> D7
- U6 pad 11: unconnected-(U6-I10/~{OE}-Pad11) -> GND
- U7 pad 1: /A0 -> A0
- U7 pad 13: /D0 -> D0
- U7 pad 2: /A1 -> A1
- U8 pad 13: /IO/D4 -> D6
- U8 pad 14: /IO/D5 -> D0
- U8 pad 17: /IO/D6 -> D3
- U8 pad 18: /IO/D7 -> D2
- U8 pad 3: /IO/D0 -> D1
- U8 pad 4: /IO/D1 -> D4
- U8 pad 7: /IO/D2 -> D7
- U8 pad 8: /IO/D3 -> D5
- U9 pad 10: /IO/D5 -> D5
- U9 pad 11: /IO/D6 -> D6
- U9 pad 12: /IO/D7 -> D7
- U9 pad 16: unconnected-(U9-STEP-Pad16) -> Net-(U9-STEP)
- U9 pad 3: /IO/A0 -> A0
- U9 pad 4: /IO/A1 -> A1
- U9 pad 5: /IO/D0 -> D0
- U9 pad 6: /IO/D1 -> D1
- U9 pad 7: /IO/D2 -> D2
- U9 pad 8: /IO/D3 -> D3
- U9 pad 9: /IO/D4 -> D4
Routing:
- net GND: track 935.8 -> 0.00 mm, vias 2 -> 0
- net +5V: track 621.8 -> 0.00 mm
- net /IO/D6: track 230.0 -> 0.00 mm, vias 1 -> 0
- net RESC\: track 223.6 -> 0.00 mm, vias 2 -> 0
- net /IO/D4: track 217.4 -> 0.00 mm, vias 2 -> 0
- net /IO/D5: track 216.5 -> 0.00 mm, vias 2 -> 0
- net RX: track 213.2 -> 0.00 mm, vias 1 -> 0
- net /IO/D7: track 211.1 -> 0.00 mm, vias 1 -> 0
- net /IO/D3: track 209.2 -> 0.00 mm, vias 2 -> 0
- net TX: track 201.0 -> 0.00 mm, vias 1 -> 0
- net /IO/D1: track 186.2 -> 0.00 mm, vias 2 -> 0
- net SIOCMD: track 177.7 -> 0.00 mm
- net /IO/D2: track 176.9 -> 0.00 mm, vias 2 -> 0
- net HALT\: track 170.3 -> 0.00 mm, vias 1 -> 0
- net SIOOUT: track 169.7 -> 0.00 mm
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